Commit message: stage1_odom

File: hardware/robot_description/urdf/robot.urdf (robot description, URDF)
Before this commit: robot robot_description, 22 links, 21 joints
Links:
- removed link breadboard_link
- removed link camera_mount_link
- removed link front_caster_link
- removed link front_caster_wheel_link
- removed link left_motor_link
- removed link left_motor_plate_link
- removed link left_wheel_link
- removed link lidar_support_link
- removed link rear_caster_link
- removed link rear_caster_wheel_link
- removed link right_motor_link
- removed link right_motor_plate_link
- removed link right_wheel_link
- removed link upper_deck_link
- link base_link: geometry collision cylinder length=0.005 radius=0.2; collision cylinder length=0.005 radius=0.2
Joints:
- removed joint breadboard_joint
- removed joint camera_mount_joint
- removed joint front_caster_joint
- removed joint front_caster_wheel_joint
- removed joint left_motor_joint
- removed joint left_motor_plate_joint
- removed joint left_wheel_joint
- removed joint lidar_support_joint
- removed joint rear_caster_joint
- removed joint rear_caster_wheel_joint
- removed joint right_motor_joint
- removed joint right_motor_plate_joint
- removed joint right_wheel_joint
- removed joint upper_deck_joint

Commit message: localization_v1

File: hardware/robot_description/urdf/robot.urdf (robot description, URDF)
Before this commit: robot robot_description, 8 links, 7 joints
Joints:
- joint laser_joint: origin xyz=0 0 0 rpy=0 0 0 -> xyz=0 0 0 rpy=0 0 3.14159265

Commit message: rviz

File: hardware/robot_description/urdf/robot.urdf (robot description, URDF)
Before this commit: robot robot_description, 8 links, 7 joints
Joints:
- joint laser_joint: origin xyz=0 0 0 rpy=0 0 3.14159265 -> xyz=0 0 0 rpy=0 0 0
